File: KittyFeeder2_PCB.kicad_pcb (KiCad board)
At the start: 2 copper layers, 114.6 x 94.7 mm, 43 parts, among them J1 ESP8266, J10 PWR_EN, J2 COOLER_PWR, J3 DHT_11, J4 SERVO_1, J5 SERVO_2, J6 GND_IN, J7 3V3_IN, J8 5V_IN, J9 12V_IN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

Commit message: Let autorouter rip
Parts:
- moved R18 2.11 mm to (166.9, 56.3)
- moved R16 1.87 mm to (173.1, 70.2), turned to 270 degrees
Routing:
- net /ESP_RST: track 0.00 -> 127.2 mm, vias 0 -> 1
- net /ESP_CH: track 0.00 -> 123.1 mm, vias 0 -> 1
- net Net-(DS1-Pad3): track 0.00 -> 102.7 mm
- net /SCL: track 0.00 -> 87.2 mm, vias 0 -> 1
- net /SERVO_2: track 0.00 -> 84.1 mm
- net /SDA: track 0.00 -> 83.6 mm, vias 0 -> 1
- net /LCD_RS: track 0.00 -> 81.8 mm
- net /LCD_EN: track 0.00 -> 78.3 mm
- net /SERVO_1: track 0.00 -> 71.1 mm, vias 0 -> 1
- net /B_LEFT: track 16.5 -> 83.5 mm
- net /LCD_D5: track 0.00 -> 66.1 mm
- net /TEMP_DATA: track 4.26 -> 69.1 mm
- net /LCD_D4: track 0.00 -> 63.5 mm, vias 0 -> 1
- net Net-(J3-Pad3): track 2.30 -> 64.2 mm, vias 0 -> 1
- net /LCD_D7: track 0.00 -> 59.3 mm
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
Commit message: passing drc
Parts:
- moved U1 8.36 mm to (120.0, 67.4), turned to 180 degrees
- moved DS1 2.50 mm to (133.2, 58.0)
- moved R18 2.25 mm to (166.9, 54.0)
Routing:
- net GND_IN: track 557.8 -> 601.4 mm, vias 3 -> 4
- net /SCL: track 87.2 -> 97.0 mm, vias 1 -> 0
- net Net-(DS1-Pad3): track 102.7 -> 94.6 mm, vias 0 -> 1
- net /LCD_D4: track 63.5 -> 70.8 mm, vias 1 -> 2
- net /SERVO_2: track 84.1 -> 90.7 mm
- net 5V_IN: track 416.6 -> 422.5 mm
- net /SDA: track 83.6 -> 87.3 mm, vias 1 -> 0
- net PWR_ENABLE: track 80.2 -> 83.7 mm
- net /LCD_EN: track 78.3 -> 80.0 mm
- net /LCD_RS: track 81.8 -> 83.3 mm
- net /LCD_D5: track 66.1 -> 67.0 mm
- net /LCD_D6: track 59.3 -> 60.2 mm
- net /LCD_D7: track 59.3 -> 60.1 mm
Other:
- board size 114.6 x 94.7 mm -> 117 x 97.2 mm
- rule pad_to_mask_clearance: 0.2 -> 0.1
